Commit message: add crazyflie 3d model

File: crazyflie_description/urdf/crazyflie.urdf.xacro (robot description, xacro)
@@ -3,6 +3,7 @@
   <link name="base_link">
     <inertial>
-      <mass value="1.477" />
+      <mass value="0.019" />
       <origin xyz="0 0 0" />
+      <!-- ToDo: This is not correct! -->
       <inertia ixx="0.01152" ixy="0.0" ixz="0.0" iyy="0.01152" iyz="0.0" izz="0.0218" />
     </inertial>
@@ -10,7 +11,8 @@
       <origin xyz="0 0 0" rpy="0 0 0" />
       <geometry>
-        <mesh filename="package://crazyflie_description/meshes/cf_model_s_revA.dae"/>
+        <mesh filename="package://crazyflie_description/meshes/crazyflie.dae"/>
       </geometry>
     </visual>
+    <!-- ToDo: insert collision model -->
   </link>
 </robot>

Commit message: added project to pycharm

File: crazyflie_description/urdf/crazyflie.urdf.xacro (robot description, xacro)
@@ -1,18 +1,18 @@
 <?xml version="1.0"?>
 <robot xmlns:xacro="http://www.ros.org/wiki/xacro" name="crazyflie">
-  <link name="base_link">
-    <inertial>
-      <mass value="0.019" />
-      <origin xyz="0 0 0" />
-      <!-- ToDo: This is not correct! -->
-      <inertia ixx="0.01152" ixy="0.0" ixz="0.0" iyy="0.01152" iyz="0.0" izz="0.0218" />
-    </inertial>
-    <visual>
-      <origin xyz="0 0 0" rpy="0 0 0" />
-      <geometry>
-        <mesh filename="package://crazyflie_description/meshes/crazyflie.dae"/>
-      </geometry>
-    </visual>
-    <!-- ToDo: insert collision model -->
-  </link>
+    <link name="base_link">
+        <inertial>
+            <mass value="0.019"/>
+            <origin xyz="0 0 0"/>
+            <!-- ToDo: This is not correct! -->
+            <inertia ixx="0.01152" ixy="0.0" ixz="0.0" iyy="0.01152" iyz="0.0" izz="0.0218"/>
+        </inertial>
+        <visual>
+            <origin xyz="0 0 0" rpy="0 0 0"/>
+            <geometry>
+                <mesh filename="package://crazyflie_description/meshes/crazyflie.dae"/>
+            </geometry>
+        </visual>
+        <!-- ToDo: insert collision model -->
+    </link>
 </robot>

File: crazyflie_description/urdf/crazyflie2.urdf.xacro (robot description, xacro)
@@ -1,21 +1,21 @@
 <?xml version="1.0"?>
 <robot xmlns:xacro="http://www.ros.org/wiki/xacro" name="crazyflie2">
-  <xacro:property name="rotor_drag_coefficient" value="1.8580e-05"/> <!-- [N.m.s^2] -->
-  <xacro:property name="moment_constant" value="0.005"/> <!-- [N.s^2] -->
-  <link name="base_link">
-    <inertial>
-      <mass value="0.027" />
-      <origin xyz="0 0 0" />
-      <!-- Refer to page 39 in http://groups.csail.mit.edu/robotics-center/public_papers/Landry15.pdf -->
-      <inertia ixx="2.3951e-5" ixy="0.0" ixz="0.0" iyy="2.3951e-5" iyz="0.0" izz="3.2347e-5" />
-      <!-- In Kg m^2 -->
-    </inertial>
-    <visual>
-      <origin xyz="0 0 0" rpy="0 0 0" />
-      <geometry>
-        <mesh filename="package://crazyflie_description/meshes/crazyflie2.dae"/>
-      </geometry>
-    </visual>
-    <!-- ToDo: insert collision model -->
-  </link>
+    <xacro:property name="rotor_drag_coefficient" value="1.8580e-05"/> <!-- [N.m.s^2] -->
+    <xacro:property name="moment_constant" value="0.005"/> <!-- [N.s^2] -->
+    <link name="base_link">
+        <inertial>
+            <mass value="0.027"/>
+            <origin xyz="0 0 0"/>
+            <!-- Refer to page 39 in http://groups.csail.mit.edu/robotics-center/public_papers/Landry15.pdf -->
+            <inertia ixx="2.3951e-5" ixy="0.0" ixz="0.0" iyy="2.3951e-5" iyz="0.0" izz="3.2347e-5"/>
+            <!-- In Kg m^2 -->
+        </inertial>
+        <visual>
+            <origin xyz="0 0 0" rpy="0 0 0"/>
+            <geometry>
+                <mesh filename="package://crazyflie_description/meshes/crazyflie2.dae"/>
+            </geometry>
+        </visual>
+        <!-- ToDo: insert collision model -->
+    </link>
 </robot>
